File: boost_regulator_simple/boost_regulator_simple.sch (KiCad schematic (older format))
At the start: 17 parts, among them Q1 MOS_N, U1 LM555N

Commit message: [boost_regulator_simple] First pass layout complete.
Parts:
- removed Q1: MOS_N, Transistors_TO-247:TO-247_Vertical_Neutral123, symbol MOS_N
- added P1, P2, P3, P4: CONN_01X01, NQBit:Screw_Terminal_x1, symbol CONN_01X01
- added Q1: MOSFET-N, Transistors_TO-247:TO-247_Vertical_Neutral123, symbol MOSFET-N
- RV1, RV2: footprint Potentiometers:Potentiometer_Trimmer-Suntan-TSR-3386C -> NQBit:Potentiometer_Thumbwheel
Connections:
- net labels added: BOOST_OUT
- wire segments 42 -> 48
Other:
- moved on the sheet: C1, D3, R3
