File: boost_regulator_simple/boost_regulator_simple.sch (KiCad schematic (older format))
At the start: 21 parts, among them P1 CONN_01X01, P2 CONN_01X01, P3 CONN_01X01, P4 CONN_01X01, Q1 MOSFET-N, U1 LM555N

Commit message: [boost_regulator_simple] Made changes to reduce EMI and other cosmetics.
Parts:
- Q1: footprint Transistors_TO-247:TO-247_Vertical_Neutral123 -> NQBit:TO-247_Vertical_Neutral123
Changed lines of the file:
@@
 LIBS:valves
 LIBS:nqbit
+LIBS:boost_regulator_simple-cache
 EELAYER 25 0
 EELAYER END
@@
 $EndComp
 $Comp
-L +9V #PWR9
+L +9V #PWR01
 U 1 1 54F13478
 P 5450 2400
-F 0 "#PWR9" H 5450 2370 20  0001 C CNN
+F 0 "#PWR01" H 5450 2370 20  0001 C CNN
 F 1 "+9V" H 5450 2510 30  0000 C CNN
 F 2 "" H 5450 2400 60  0000 C CNN
@@
 $EndComp
 $Comp
-L GND #PWR10
+L GND #PWR02
 U 1 1 54F13BB5
 P 5450 3600
-F 0 "#PWR10" H 5450 3600 30  0001 C CNN
+F 0 "#PWR02" H 5450 3600 30  0001 C CNN
 F 1 "GND" H 5450 3530 30  0001 C CNN
 F 2 "" H 5450 3600 60  0000 C CNN
@@
 $EndComp
 $Comp
-L GND #PWR11
+L GND #PWR03
 U 1 1 54F13DC9
 P 6150 3600
-F 0 "#PWR11" H 6150 3600 30  0001 C CNN
+F 0 "#PWR03" H 6150 3600 30  0001 C CNN
 F 1 "GND" H 6150 3530 30  0001 C CNN
 F 2 "" H 6150 3600 60  0000 C CNN
@@
 $EndComp
 $Comp
-L GND #PWR8
+L GND #PWR04
 U 1 1 54F14811
 P 5100 2900
-F 0 "#PWR8" H 5100 2900 30  0001 C CNN
+F 0 "#PWR04" H 5100 2900 30  0001 C CNN
 F 1 "GND" H 5100 2830 30  0001 C CNN
 F 2 "" H 5100 2900 60  0000 C CNN
@@
 $EndComp
 $Comp
-L GND #PWR6
+L GND #PWR05
 U 1 1 54F15F8B
 P 3150 1650
-F 0 "#PWR6" H 3150 1650 30  0001 C CNN
+F 0 "#PWR05" H 3150 1650 30  0001 C CNN
 F 1 "GND" H 3150 1580 30  0001 C CNN
 F 2 "" H 3150 1650 60  0000 C CNN
@@
 $EndComp
 $Comp
-L +9V #PWR1
+L +9V #PWR06
 U 1 1 54F18F43
 P 2100 1050
-F 0 "#PWR1" H 2100 1020 20  0001 C CNN
+F 0 "#PWR06" H 2100 1020 20  0001 C CNN
 F 1 "+9V" V 2100 1200 30  0000 C CNN
 F 2 "" H 2100 1050 60  0000 C CNN
@@
 $EndComp
 $Comp
-L VCC #PWR2
+L VCC #PWR07
 U 1 1 54F18F83
 P 2250 1050
-F 0 "#PWR2" H 2250 1150 30  0001 C CNN
+F 0 "#PWR07" H 2250 1150 30  0001 C CNN
 F 1 "VCC" V 2250 1200 30  0000 C CNN
 F 2 "" H 2250 1050 60  0000 C CNN
@@
 $EndComp
 $Comp
-L VCC #PWR5
+L VCC #PWR08
 U 1 1 54F19502
 P 3050 1150
-F 0 "#PWR5" H 3050 1250 30  0001 C CNN
+F 0 "#PWR08" H 3050 1250 30  0001 C CNN
 F 1 "VCC" V 3050 1300 30  0000 C CNN
 F 2 "" H 3050 1150 60  0000 C CNN
@@
 $EndComp
 $Comp
-L GND #PWR12
+L GND #PWR09
 U 1 1 54F19C09
 P 6500 2250
-F 0 "#PWR12" H 6500 2250 30  0001 C CNN
+F 0 "#PWR09" H 6500 2250 30  0001 C CNN
 F 1 "GND" H 6500 2180 30  0001 C CNN
 F 2 "" H 6500 2250 60  0000 C CNN
@@
 $EndComp
 $Comp
-L GND #PWR7
+L GND #PWR010
 U 1 1 54F19CE0
 P 3750 4050
-F 0 "#PWR7" H 3750 4050 30  0001 C CNN
+F 0 "#PWR010" H 3750 4050 30  0001 C CNN
 F 1 "GND" H 3750 3980 30  0001 C CNN
 F 2 "" H 3750 4050 60  0000 C CNN
@@
 $EndComp
 $Comp
-L GND #PWR13
+L GND #PWR011
 U 1 1 54F23D47
 P 6550 3350
-F 0 "#PWR13" H 6550 3350 30  0001 C CNN
+F 0 "#PWR011" H 6550 3350 30  0001 C CNN
 F 1 "GND" H 6550 3280 30  0001 C CNN
 F 2 "" H 6550 3350 60  0000 C CNN
@@
 $EndComp
 $Comp
-L VCC #PWR3
+L VCC #PWR012
 U 1 1 54F26F4D
 P 2600 1400
-F 0 "#PWR3" H 2600 1500 30  0001 C CNN
+F 0 "#PWR012" H 2600 1500 30  0001 C CNN
 F 1 "VCC" V 2600 1550 30  0000 C CNN
 F 2 "" H 2600 1400 60  0000 C CNN
@@
 $EndComp
 $Comp
-L GND #PWR4
+L GND #PWR013
 U 1 1 54F26F6B
 P 2600 1700
-F 0 "#PWR4" H 2600 1700 30  0001 C CNN
+F 0 "#PWR013" H 2600 1700 30  0001 C CNN
 F 1 "GND" H 2600 1630 30  0001 C CNN
 F 2 "" H 2600 1700 60  0000 C CNN
@@
 F 0 "Q1" H 5350 3201 40  0000 R CNN
 F 1 "MOSFET-N" H 5850 3300 40  0000 R CNN
-F 2 "Transistors_TO-247:TO-247_Vertical_Neutral123" H 5650 3350 29  0001 C CNN
+F 2 "NQBit:TO-247_Vertical_Neutral123" H 5650 3350 29  0001 C CNN
 F 3 "http://www.digikey.com/product-detail/en/C2M1000170D/C2M1000170D-ND/4399776" H 5650 3500 60  0001 C CNN
 	1    5350 3350

Commit message: [boost_regulator_simple] Added more filter caps to U1 and the inductor.
Parts:
- added C? (x2): 0.01uF, Capacitors_ThroughHole:Capacitor3MMDiscRM2.5, symbol C
Connections:
- wire segments 48 -> 51
Changed lines of the file:
@@
 L +9V #PWR06
 U 1 1 54F18F43
-P 2100 1050
-F 0 "#PWR06" H 2100 1020 20  0001 C CNN
-F 1 "+9V" V 2100 1200 30  0000 C CNN
-F 2 "" H 2100 1050 60  0000 C CNN
-F 3 "" H 2100 1050 60  0000 C CNN
-	1    2100 1050
+P 1850 1200
+F 0 "#PWR06" H 1850 1170 20  0001 C CNN
+F 1 "+9V" V 1850 1350 30  0000 C CNN
+F 2 "" H 1850 1200 60  0000 C CNN
+F 3 "" H 1850 1200 60  0000 C CNN
+	1    1850 1200
 	0    -1   -1   0
 $EndComp
@@
 L VCC #PWR07
 U 1 1 54F18F83
-P 2250 1050
-F 0 "#PWR07" H 2250 1150 30  0001 C CNN
-F 1 "VCC" V 2250 1200 30  0000 C CNN
-F 2 "" H 2250 1050 60  0000 C CNN
-F 3 "" H 2250 1050 60  0000 C CNN
-	1    2250 1050
+P 2000 1200
+F 0 "#PWR07" H 2000 1300 30  0001 C CNN
+F 1 "VCC" V 2000 1350 30  0000 C CNN
+F 2 "" H 2000 1200 60  0000 C CNN
+F 3 "" H 2000 1200 60  0000 C CNN
+	1    2000 1200
 	0    1    1    0
 $EndComp
@@
 	6150 3100 6150 3150
 Wire Wire Line
-	5450 2450 5100 2450
+	4800 2450 5450 2450
 Wire Wire Line
 	5100 2850 5100 2900
@@
 Connection ~ 4050 1150
 Wire Wire Line
-	2100 1050 2250 1050
+	1850 1200 2000 1200
 Wire Wire Line
 	6500 1800 6500 1700
@@
 Wire Wire Line
 	4600 3200 4600 3400
+$Comp
+L C C?
+U 1 1 54F2B6B2
+P 1900 1450
+F 0 "C?" H 1900 1550 40  0000 L CNN
+F 1 "0.01uF" H 1906 1365 40  0000 L CNN
+F 2 "Capacitors_ThroughHole:Capacitor3MMDiscRM2.5" H 1938 1300 30  0001 C CNN
+F 3 "" H 1900 1450 60  0000 C CNN
+	1    1900 1450
+	1    0    0    -1
+$EndComp
+$Comp
+L GND #PWR?
+U 1 1 54F2BE24
+P 1900 1700
+F 0 "#PWR?" H 1900 1700 30  0001 C CNN
+F 1 "GND" H 1900 1630 30  0001 C CNN
+F 2 "" H 1900 1700 60  0000 C CNN
+F 3 "" H 1900 1700 60  0000 C CNN
+	1    1900 1700
+	1    0    0    -1
+$EndComp
+Wire Wire Line
+	1900 1700 1900 1650
+Wire Wire Line
+	1900 1250 1900 1200
+Connection ~ 1900 1200
+$Comp
+L C C?
+U 1 1 54F2CB72
+P 4800 2650
+F 0 "C?" H 4800 2750 40  0000 L CNN
+F 1 "0.01uF" H 4806 2565 40  0000 L CNN
+F 2 "Capacitors_ThroughHole:Capacitor3MMDiscRM2.5" H 4838 2500 30  0001 C CNN
+F 3 "" H 4800 2650 60  0000 C CNN
+	1    4800 2650
+	1    0    0    -1
+$EndComp
+Connection ~ 5100 2450
+Wire Wire Line
+	4800 2850 5100 2850
 $EndSCHEMATC

Commit message: [boost_regulator_simple] Off to fab!
Parts:
- gave numbers to parts that had none: 2
Changed lines of the file:
@@
 $EndComp
 $Comp
-L +9V #PWR01
+L +9V #PWR10
 U 1 1 54F13478
 P 5450 2400
-F 0 "#PWR01" H 5450 2370 20  0001 C CNN
+F 0 "#PWR10" H 5450 2370 20  0001 C CNN
 F 1 "+9V" H 5450 2510 30  0000 C CNN
 F 2 "" H 5450 2400 60  0000 C CNN
@@
 $EndComp
 $Comp
-L GND #PWR02
+L GND #PWR11
 U 1 1 54F13BB5
 P 5450 3600
-F 0 "#PWR02" H 5450 3600 30  0001 C CNN
+F 0 "#PWR11" H 5450 3600 30  0001 C CNN
 F 1 "GND" H 5450 3530 30  0001 C CNN
 F 2 "" H 5450 3600 60  0000 C CNN
@@
 $EndComp
 $Comp
-L GND #PWR03
+L GND #PWR12
 U 1 1 54F13DC9
 P 6150 3600
-F 0 "#PWR03" H 6150 3600 30  0001 C CNN
+F 0 "#PWR12" H 6150 3600 30  0001 C CNN
 F 1 "GND" H 6150 3530 30  0001 C CNN
 F 2 "" H 6150 3600 60  0000 C CNN
@@
 $EndComp
 $Comp
-L GND #PWR04
+L GND #PWR9
 U 1 1 54F14811
 P 5100 2900
-F 0 "#PWR04" H 5100 2900 30  0001 C CNN
+F 0 "#PWR9" H 5100 2900 30  0001 C CNN
 F 1 "GND" H 5100 2830 30  0001 C CNN
 F 2 "" H 5100 2900 60  0000 C CNN
@@
 $EndComp
 $Comp
-L GND #PWR05
+L GND #PWR7
 U 1 1 54F15F8B
 P 3150 1650
-F 0 "#PWR05" H 3150 1650 30  0001 C CNN
+F 0 "#PWR7" H 3150 1650 30  0001 C CNN
 F 1 "GND" H 3150 1580 30  0001 C CNN
 F 2 "" H 3150 1650 60  0000 C CNN
@@
 $EndComp
 $Comp
-L +9V #PWR06
+L +9V #PWR1
 U 1 1 54F18F43
 P 1850 1200
-F 0 "#PWR06" H 1850 1170 20  0001 C CNN
+F 0 "#PWR1" H 1850 1170 20  0001 C CNN
 F 1 "+9V" V 1850 1350 30  0000 C CNN
 F 2 "" H 1850 1200 60  0000 C CNN
@@
 $EndComp
 $Comp
-L VCC #PWR07
+L VCC #PWR3
 U 1 1 54F18F83
 P 2000 1200
-F 0 "#PWR07" H 2000 1300 30  0001 C CNN
+F 0 "#PWR3" H 2000 1300 30  0001 C CNN
 F 1 "VCC" V 2000 1350 30  0000 C CNN
 F 2 "" H 2000 1200 60  0000 C CNN
@@
 $EndComp
 $Comp
-L VCC #PWR08
+L VCC #PWR6
 U 1 1 54F19502
 P 3050 1150
-F 0 "#PWR08" H 3050 1250 30  0001 C CNN
+F 0 "#PWR6" H 3050 1250 30  0001 C CNN
 F 1 "VCC" V 3050 1300 30  0000 C CNN
 F 2 "" H 3050 1150 60  0000 C CNN
@@
 $EndComp
 $Comp
-L GND #PWR09
+L GND #PWR13
 U 1 1 54F19C09
 P 6500 2250
-F 0 "#PWR09" H 6500 2250 30  0001 C CNN
+F 0 "#PWR13" H 6500 2250 30  0001 C CNN
 F 1 "GND" H 6500 2180 30  0001 C CNN
 F 2 "" H 6500 2250 60  0000 C CNN
@@
 $EndComp
 $Comp
-L GND #PWR010
+L GND #PWR8
 U 1 1 54F19CE0
 P 3750 4050
-F 0 "#PWR010" H 3750 4050 30  0001 C CNN
+F 0 "#PWR8" H 3750 4050 30  0001 C CNN
 F 1 "GND" H 3750 3980 30  0001 C CNN
 F 2 "" H 3750 4050 60  0000 C CNN
@@
 $EndComp
 $Comp
-L GND #PWR011
+L GND #PWR14
 U 1 1 54F23D47
 P 6550 3350
-F 0 "#PWR011" H 6550 3350 30  0001 C CNN
+F 0 "#PWR14" H 6550 3350 30  0001 C CNN
 F 1 "GND" H 6550 3280 30  0001 C CNN
 F 2 "" H 6550 3350 60  0000 C CNN
@@
 $EndComp
 $Comp
-L VCC #PWR012
+L VCC #PWR4
 U 1 1 54F26F4D
 P 2600 1400
-F 0 "#PWR012" H 2600 1500 30  0001 C CNN
+F 0 "#PWR4" H 2600 1500 30  0001 C CNN
 F 1 "VCC" V 2600 1550 30  0000 C CNN
 F 2 "" H 2600 1400 60  0000 C CNN
@@
 $EndComp
 $Comp
-L GND #PWR013
+L GND #PWR5
 U 1 1 54F26F6B
 P 2600 1700
-F 0 "#PWR013" H 2600 1700 30  0001 C CNN
+F 0 "#PWR5" H 2600 1700 30  0001 C CNN
 F 1 "GND" H 2600 1630 30  0001 C CNN
 F 2 "" H 2600 1700 60  0000 C CNN
@@
 	4600 3200 4600 3400
 $Comp
-L C C?
+L C C6
 U 1 1 54F2B6B2
 P 1900 1450
-F 0 "C?" H 1900 1550 40  0000 L CNN
+F 0 "C6" H 1900 1550 40  0000 L CNN
 F 1 "0.01uF" H 1906 1365 40  0000 L CNN
 F 2 "Capacitors_ThroughHole:Capacitor3MMDiscRM2.5" H 1938 1300 30  0001 C CNN
@@
 $EndComp
 $Comp
-L GND #PWR?
+L GND #PWR2
 U 1 1 54F2BE24
 P 1900 1700
-F 0 "#PWR?" H 1900 1700 30  0001 C CNN
+F 0 "#PWR2" H 1900 1700 30  0001 C CNN
 F 1 "GND" H 1900 1630 30  0001 C CNN
 F 2 "" H 1900 1700 60  0000 C CNN
@@
 Connection ~ 1900 1200
 $Comp
-L C C?
+L C C7
 U 1 1 54F2CB72
 P 4800 2650
-F 0 "C?" H 4800 2750 40  0000 L CNN
+F 0 "C7" H 4800 2750 40  0000 L CNN
 F 1 "0.01uF" H 4806 2565 40  0000 L CNN
 F 2 "Capacitors_ThroughHole:Capacitor3MMDiscRM2.5" H 4838 2500 30  0001 C CNN
