File: boost_regulator_simple/boost_regulator_simple.kicad_pcb (KiCad board)
At the start: 2 copper layers, 61 x 53.3 mm, 21 parts, among them P1 CONN_01X01, P2 CONN_01X01, P3 CONN_01X01, P4 CONN_01X01, Q1 MOSFET-N, U1 LM555N

Commit message: [boost_regulator_simple] Off to fab!
Parts:
- added C6: 0.01uF, Capacitors_ThroughHole:Capacitor3MMDiscRM2.5, F.Cu at (115.6, 65.4)
- added C7: 0.01uF, Capacitors_ThroughHole:Capacitor3MMDiscRM2.5, F.Cu at (112.4, 88.9)
- moved C1 1.27 mm to (118.1, 58.4)
Routing:
- net VCC: track 63.5 -> 66.7 mm
Other:
- board text added: "Boosty V0.1"
- board text added: "Designed by Nathaniel with help from Mark"
Changed lines of the file:
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@@
 (kicad_pcb (version 4) (host pcbnew 0.201502181246+5430~21~ubuntu14.04.1-product)
   (general
-    (links 45)
+    (links 49)
     (no_connects 0)
-    (area 71.161001 52.019999 142.589011 105.460001)
+    (area 79.959999 52.019999 141.020001 105.460001)
     (thickness 1.6)
-    (drawings 4)
-    (tracks 37)
+    (drawings 12)
+    (tracks 39)
     (zones 0)
-    (modules 21)
+    (modules 23)
     (nets 15)
   )
@@
     (pad_to_mask_clearance 0)
     (aux_axis_origin 0 0)
-    (visible_elements FFFFFF7F)
+    (visible_elements FFFEFF7F)
     (pcbplotparams
       (layerselection 0x010f0_80000001)
@@
       (psa4output false)
       (plotreference true)
-      (plotvalue true)
+      (plotvalue false)
       (plotinvisibletext false)
       (padsonsilk false)
@@
   )
   (module Capacitors_Elko_ThroughHole:Elko_vert_20x10mm_RM5 (layer F.Cu)
-    (at 118.11 59.69 180)
+    (at 118.11 58.42 180)
     (descr "Electrolytic Capacitor, vertical, diameter 10mm, RM 5mm, radial,")
     (tags "Electrolytic Capacitor, vertical, diameter 10mm, RM 5mm, Elko, Electrolytkondensator, Kondensator gepolt, Durchmesser 10mm, radial,")
@@
     (descr "8 pins DIL package, round pads")
     (tags DIL)
-    (fp_text reference U1 (at -6.35 0 360) (layer F.SilkS)
+    (fp_text reference U1 (at 6.35 0 360) (layer F.SilkS)
       (effects (font (size 1 1) (thickness 0.15)))
     )
@@
       (net 1 GND))
   )
+  (module Capacitors_ThroughHole:Capacitor3MMDiscRM2.5 (layer F.Cu)
+    (at 115.57 65.405 180)
+    (descr Capacitor3MMDiscRM2.5)
+    (tags C)
+    (fp_text reference C6 (at 3.81 0 180) (layer F.SilkS)
+      (effects (font (size 1 1) (thickness 0.15)))
+    )
+    (fp_text value 0.01uF (at 0 -2.286 180) (layer F.SilkS) hide
+      (effects (font (size 1 1) (thickness 0.15)))
+    )
+    (fp_line (start -2.4892 -1.27) (end 2.54 -1.27) (layer F.SilkS) (width 0.15))
+    (fp_line (start 2.54 -1.27) (end 2.54 1.27) (layer F.SilkS) (width 0.15))
+    (fp_line (start 2.54 1.27) (end -2.54 1.27) (layer F.SilkS) (width 0.15))
+    (fp_line (start -2.54 1.27) (end -2.54 -1.27) (layer F.SilkS) (width 0.15))
+    (fp_line (start -2.54 -0.635) (end -1.905 -1.27) (layer F.SilkS) (width 0.15))
+    (pad 1 thru_hole circle (at -1.27 0 180) (size 1.50114 1.50114) (drill 0.8001) (layers *.Cu *.Mask F.SilkS)
+      (net 2 VCC))
+    (pad 2 thru_hole circle (at 1.27 0 180) (size 1.50114 1.50114) (drill 0.8001) (layers *.Cu *.Mask F.SilkS)
+      (net 1 GND))
+    (model Capacitors_ThroughHole/Capacitor3MMDiscRM2.5.wrl
+      (at (xyz 0 0 0))
+      (scale (xyz 1 1 1))
+      (rotate (xyz 0 0 0))
+    )
+  )
+  (module Capacitors_ThroughHole:Capacitor3MMDiscRM2.5 (layer F.Cu)
+    (at 112.395 88.9)
+    (descr Capacitor3MMDiscRM2.5)
+    (tags C)
+    (fp_text reference C7 (at 3.81 0 90) (layer F.SilkS)
+      (effects (font (size 1 1) (thickness 0.15)))
+    )
+    (fp_text value 0.01uF (at 0 -2.286) (layer F.SilkS) hide
+      (effects (font (size 1 1) (thickness 0.15)))
+    )
+    (fp_line (start -2.4892 -1.27) (end 2.54 -1.27) (layer F.SilkS) (width 0.15))
+    (fp_line (start 2.54 -1.27) (end 2.54 1.27) (layer F.SilkS) (width 0.15))
+    (fp_line (start 2.54 1.27) (end -2.54 1.27) (layer F.SilkS) (width 0.15))
+    (fp_line (start -2.54 1.27) (end -2.54 -1.27) (layer F.SilkS) (width 0.15))
+    (fp_line (start -2.54 -0.635) (end -1.905 -1.27) (layer F.SilkS) (width 0.15))
+    (pad 1 thru_hole circle (at -1.27 0) (size 1.50114 1.50114) (drill 0.8001) (layers *.Cu *.Mask F.SilkS)
+      (net 2 VCC))
+    (pad 2 thru_hole circle (at 1.27 0) (size 1.50114 1.50114) (drill 0.8001) (layers *.Cu *.Mask F.SilkS)
+      (net 1 GND))
+    (model Capacitors_ThroughHole/Capacitor3MMDiscRM2.5.wrl
+      (at (xyz 0 0 0))
+      (scale (xyz 1 1 1))
+      (rotate (xyz 0 0 0))
+    )
+  )
+  (gr_text "Boosty V0.1" (at 102.362 62.865) (layer F.SilkS)
+    (effects (font (size 1.5 1.5) (thickness 0.3)))
+  )
+  (gr_line (start 101.473 59.182) (end 104.013 57.912) (layer F.SilkS) (width 0.2))
+  (gr_text "Designed by Nathaniel\nwith help from Mark" (at 83.82 78.74 90) (layer F.SilkS)
+    (effects (font (size 1.5 1.5) (thickness 0.3)))
+  )
+  (gr_circle (center 102.997 56.896) (end 103.251 57.15) (layer F.SilkS) (width 0.2))
+  (gr_circle (center 101.6 57.023) (end 102.235 57.404) (layer F.SilkS) (width 0.2))
+  (gr_arc (start 105.156 56.515) (end 103.632 55.88) (angle 81.4163701) (layer F.SilkS) (width 0.2))
+  (gr_arc (start 97.536 57.023) (end 100.711 56.007) (angle -34.05673509) (layer F.SilkS) (width 0.2))
+  (gr_circle (center 102.362 58.166) (end 101.727 60.706) (layer F.SilkS) (width 0.2))
   (gr_line (start 140.97 105.41) (end 140.97 52.07) (layer Edge.Cuts) (width 0.1))
   (gr_line (start 80.01 105.41) (end 140.97 105.41) (layer Edge.Cuts) (width 0.1))
@@
   (segment (start 115.57 93.98) (end 118.15 96.56) (width 2.54) (layer F.Cu) (net 2) (status 10))
   (segment (start 118.15 96.56) (end 129.845 96.56) (width 2.54) (layer F.Cu) (net 2) (status 20))
-  (segment (start 123.19 64.77) (end 118.11 59.69) (width 1.27) (layer F.Cu) (net 2))
-  (segment (start 123.19 66.04) (end 123.19 64.77) (width 1.27) (layer F.Cu) (net 2))
+  (segment (start 119.38 67.945) (end 116.84 65.405) (width 1.27) (layer F.Cu) (net 2))
+  (segment (start 119.38 68.58) (end 119.38 67.945) (width 1.27) (layer F.Cu) (net 2))
+  (segment (start 116.84 59.69) (end 118.11 58.42) (width 1.27) (layer F.Cu) (net 2))
+  (segment (start 116.84 65.405) (end 116.84 59.69) (width 1.27) (layer F.Cu) (net 2))
   (segment (start 133.35 82.55) (end 134.62 83.82) (width 1.27) (layer F.Cu) (net 3) (status 20))
   (segment (start 133.35 78.74) (end 133.35 82.55) (width 1.27) (layer F.Cu) (net 3) (status 10))
@@
     (connect_pads (clearance 0.508))
     (min_thickness 0.254)
-    (fill (arc_segments 16) (thermal_gap 0.508) (thermal_bridge_width 0.508))
+    (fill yes (arc_segments 16) (thermal_gap 0.508) (thermal_bridge_width 0.508))
     (polygon
       (pts
@@
     (connect_pads (clearance 0.508))
     (min_thickness 0.254)
-    (fill (arc_segments 16) (thermal_gap 0.508) (thermal_bridge_width 0.508))
+    (fill yes (arc_segments 16) (thermal_gap 0.508) (thermal_bridge_width 0.508))
     (polygon
       (pts
@@
     (connect_pads yes (clearance 0.508))
     (min_thickness 0.254)
-    (fill (arc_segments 16) (thermal_gap 0.508) (thermal_bridge_width 0.508))
+    (fill yes (arc_segments 16) (thermal_gap 0.508) (thermal_bridge_width 0.508))
     (polygon
       (pts
@@
     (connect_pads yes (clearance 0.508))
     (min_thickness 0.254)
-    (fill (arc_segments 16) (thermal_gap 0.508) (thermal_bridge_width 0.508))
+    (fill yes (arc_segments 16) (thermal_gap 0.508) (thermal_bridge_width 0.508))
     (polygon
       (pts
@@
     (connect_pads yes (clearance 0.508))
     (min_thickness 0.254)
-    (fill (arc_segments 16) (thermal_gap 0.508) (thermal_bridge_width 0.508))
+    (fill yes (arc_segments 16) (thermal_gap 0.508) (thermal_bridge_width 0.508))
     (polygon
       (pts

Commit message: [boost_regulator_simple] Added full part datasheets and regenerated gerbers and schematic.
Parts:
- moved P4 1.27 mm to (86.4, 58.4)
Other:
- board size 61 x 53.3 mm -> 66 x 53.3 mm
Changed lines of the file:
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@@
     (links 49)
     (no_connects 0)
-    (area 79.959999 52.019999 141.020001 105.460001)
+    (area 71.161001 52.019999 142.925001 105.460001)
     (thickness 1.6)
     (drawings 12)
@@
   )
   (module NQBit:Screw_Terminal_x1 (layer F.Cu)
-    (at 87.63 58.42 90)
+    (at 86.36 58.42 90)
     (descr http://www.digikey.com/product-detail/en/7693/7693K-ND/151562)
     (fp_text reference P4 (at -6.35 0 180) (layer F.SilkS)
@@
   (gr_arc (start 97.536 57.023) (end 100.711 56.007) (angle -34.05673509) (layer F.SilkS) (width 0.2))
   (gr_circle (center 102.362 58.166) (end 101.727 60.706) (layer F.SilkS) (width 0.2))
-  (gr_line (start 140.97 105.41) (end 140.97 52.07) (layer Edge.Cuts) (width 0.1))
-  (gr_line (start 80.01 105.41) (end 140.97 105.41) (layer Edge.Cuts) (width 0.1))
-  (gr_line (start 80.01 52.07) (end 80.01 105.41) (layer Edge.Cuts) (width 0.1))
-  (gr_line (start 140.97 52.07) (end 80.01 52.07) (layer Edge.Cuts) (width 0.1))
+  (gr_line (start 142.875 105.41) (end 142.875 52.07) (layer Edge.Cuts) (width 0.1))
+  (gr_line (start 76.835 105.41) (end 142.875 105.41) (layer Edge.Cuts) (width 0.1))
+  (gr_line (start 76.835 52.07) (end 76.835 105.41) (layer Edge.Cuts) (width 0.1))
+  (gr_line (start 142.875 52.07) (end 76.835 52.07) (layer Edge.Cuts) (width 0.1))
+  (segment (start 116.84 65.405) (end 116.84 59.69) (width 1.27) (layer F.Cu) (net 2))
+  (segment (start 116.84 59.69) (end 118.11 58.42) (width 1.27) (layer F.Cu) (net 2))
+  (segment (start 119.38 68.58) (end 119.38 67.945) (width 1.27) (layer F.Cu) (net 2))
+  (segment (start 119.38 67.945) (end 116.84 65.405) (width 1.27) (layer F.Cu) (net 2))
+  (segment (start 118.15 96.56) (end 129.845 96.56) (width 2.54) (layer F.Cu) (net 2) (status 20))
+  (segment (start 115.57 93.98) (end 118.15 96.56) (width 2.54) (layer F.Cu) (net 2) (status 10))
+  (segment (start 129.845 96.56) (end 136.855 96.56) (width 2.54) (layer F.Cu) (net 2) (status 30))
+  (segment (start 136.855 101.56) (end 136.855 96.56) (width 2.54) (layer F.Cu) (net 2) (status 30))
+  (segment (start 129.845 101.56) (end 136.855 101.56) (width 2.54) (layer F.Cu) (net 2) (status 30))
+  (segment (start 129.845 101.56) (end 129.845 96.56) (width 2.54) (layer F.Cu) (net 2) (status 30))
+  (segment (start 120.65 68.58) (end 123.19 66.04) (width 1.27) (layer F.Cu) (net 2) (status 20))
+  (segment (start 119.38 68.58) (end 120.65 68.58) (width 1.27) (layer F.Cu) (net 2) (status 10))
   (segment (start 111.76 76.2) (end 119.38 68.58) (width 1.27) (layer F.Cu) (net 2) (status 30))
-  (segment (start 119.38 68.58) (end 120.65 68.58) (width 1.27) (layer F.Cu) (net 2) (status 10))
-  (segment (start 120.65 68.58) (end 123.19 66.04) (width 1.27) (layer F.Cu) (net 2) (status 20))
-  (segment (start 129.845 101.56) (end 129.845 96.56) (width 2.54) (layer F.Cu) (net 2) (status 30))
-  (segment (start 129.845 101.56) (end 136.855 101.56) (width 2.54) (layer F.Cu) (net 2) (status 30))
-  (segment (start 136.855 101.56) (end 136.855 96.56) (width 2.54) (layer F.Cu) (net 2) (status 30))
-  (segment (start 129.845 96.56) (end 136.855 96.56) (width 2.54) (layer F.Cu) (net 2) (status 30))
-  (segment (start 115.57 93.98) (end 118.15 96.56) (width 2.54) (layer F.Cu) (net 2) (status 10))
-  (segment (start 118.15 96.56) (end 129.845 96.56) (width 2.54) (layer F.Cu) (net 2) (status 20))
-  (segment (start 119.38 67.945) (end 116.84 65.405) (width 1.27) (layer F.Cu) (net 2))
-  (segment (start 119.38 68.58) (end 119.38 67.945) (width 1.27) (layer F.Cu) (net 2))
-  (segment (start 116.84 59.69) (end 118.11 58.42) (width 1.27) (layer F.Cu) (net 2))
-  (segment (start 116.84 65.405) (end 116.84 59.69) (width 1.27) (layer F.Cu) (net 2))
+  (segment (start 133.35 78.74) (end 133.35 82.55) (width 1.27) (layer F.Cu) (net 3) (status 10))
   (segment (start 133.35 82.55) (end 134.62 83.82) (width 1.27) (layer F.Cu) (net 3) (status 20))
-  (segment (start 133.35 78.74) (end 133.35 82.55) (width 1.27) (layer F.Cu) (net 3) (status 10))
   (segment (start 119.38 81.28) (end 119.38 76.2) (width 1.27) (layer F.Cu) (net 4) (status 30))
+  (segment (start 119.38 71.12) (end 123.19 74.93) (width 1.27) (layer F.Cu) (net 5) (status 10))
+  (segment (start 123.19 74.93) (end 123.19 76.2) (width 1.27) (layer F.Cu) (net 5) (status 20))
+  (segment (start 123.19 76.2) (end 127 76.2) (width 1.27) (layer F.Cu) (net 5) (status 30))
   (segment (start 123.19 81.28) (end 123.19 76.2) (width 1.27) (layer F.Cu) (net 5) (status 30))
-  (segment (start 123.19 76.2) (end 127 76.2) (width 1.27) (layer F.Cu) (net 5) (status 30))
-  (segment (start 123.19 74.93) (end 123.19 76.2) (width 1.27) (layer F.Cu) (net 5) (status 20))
-  (segment (start 119.38 71.12) (end 123.19 74.93) (width 1.27) (layer F.Cu) (net 5) (status 10))
+  (segment (start 127 66.04) (end 132.08 66.04) (width 1.27) (layer F.Cu) (net 6) (status 10))
   (segment (start 132.08 66.04) (end 134.62 68.58) (width 1.27) (layer F.Cu) (net 6) (status 20))
-  (segment (start 127 66.04) (end 132.08 66.04) (width 1.27) (layer F.Cu) (net 6) (status 10))
   (segment (start 127 81.28) (end 134.62 73.66) (width 1.27) (layer F.Cu) (net 7) (status 30))
   (segment (start 127 91.44) (end 123.19 91.44) (width 1.27) (layer F.Cu) (net 8) (status 30))
+  (segment (start 106.68 68.58) (end 106.68 73.66) (width 1.27) (layer F.Cu) (net 9) (status 30))
   (segment (start 106.68 73.66) (end 111.76 73.66) (width 1.27) (layer F.Cu) (net 9) (status 30))
-  (segment (start 106.68 68.58) (end 106.68 73.66) (width 1.27) (layer F.Cu) (net 9) (status 30))
+  (segment (start 134.62 71.12) (end 138.43 74.93) (width 1.27) (layer F.Cu) (net 10) (status 10))
+  (segment (start 138.43 74.93) (end 138.43 85.09) (width 1.27) (layer F.Cu) (net 10))
   (segment (start 138.43 85.09) (end 134.62 88.9) (width 1.27) (layer F.Cu) (net 10) (status 20))
-  (segment (start 138.43 74.93) (end 138.43 85.09) (width 1.27) (layer F.Cu) (net 10))
-  (segment (start 134.62 71.12) (end 138.43 74.93) (width 1.27) (layer F.Cu) (net 10) (status 10))
+  (segment (start 134.62 86.36) (end 131.428491 83.168491) (width 1.27) (layer F.Cu) (net 11) (status 10))
+  (segment (start 131.428491 83.168491) (end 122.283523 83.168491) (width 1.27) (layer F.Cu) (net 11))
+  (segment (start 121.301509 75.581509) (end 119.38 73.66) (width 1.27) (layer F.Cu) (net 11) (status 20))
+  (segment (start 122.283523 83.168491) (end 121.301509 82.186477) (width 1.27) (layer F.Cu) (net 11))
+  (segment (start 121.301509 82.186477) (end 121.301509 75.581509) (width 1.27) (layer F.Cu) (net 11))
+  (segment (start 116.84 71.12) (end 119.38 73.66) (width 1.27) (layer B.Cu) (net 11) (status 20))
   (segment (start 111.76 71.12) (end 116.84 71.12) (width 1.27) (layer B.Cu) (net 11) (status 10))
-  (segment (start 116.84 71.12) (end 119.38 73.66) (width 1.27) (layer B.Cu) (net 11) (status 20))
-  (segment (start 121.301509 82.186477) (end 121.301509 75.581509) (width 1.27) (layer F.Cu) (net 11))
-  (segment (start 122.283523 83.168491) (end 121.301509 82.186477) (width 1.27) (layer F.Cu) (net 11))
-  (segment (start 121.301509 75.581509) (end 119.38 73.66) (width 1.27) (layer F.Cu) (net 11) (status 20))
-  (segment (start 131.428491 83.168491) (end 122.283523 83.168491) (width 1.27) (layer F.Cu) (net 11))
-  (segment (start 134.62 86.36) (end 131.428491 83.168491) (width 1.27) (layer F.Cu) (net 11) (status 10))
+  (segment (start 96.647 73.787) (end 96.52 73.66) (width 1.27) (layer F.Cu) (net 13))
+  (segment (start 96.647 79.375) (end 96.647 73.787) (width 1.27) (layer F.Cu) (net 13))
   (segment (start 96.52 68.58) (end 96.52 73.66) (width 1.27) (layer F.Cu) (net 13))
-  (segment (start 96.647 79.375) (end 96.647 73.787) (width 1.27) (layer F.Cu) (net 13))
-  (segment (start 96.647 73.787) (end 96.52 73.66) (width 1.27) (layer F.Cu) (net 13))
   (zone (net 1) (net_name GND) (layer B.Cu) (hatch edge 0.508)
     (connect_pads (clearance 0.508))
@@
     (polygon
       (pts
-        (xy 81.28 53.34) (xy 139.7 53.34) (xy 139.7 104.14) (xy 113.03 104.14) (xy 107.442 104.14)
-        (xy 105.41 102.108) (xy 105.41 74.93) (xy 104.14 73.66) (xy 83.82 73.66) (xy 81.28 71.12)
+        (xy 78.105 53.34) (xy 141.605 53.34) (xy 141.605 104.14) (xy 113.03 104.14) (xy 107.442 104.14)
+        (xy 105.41 102.108) (xy 105.41 74.93) (xy 104.14 73.66) (xy 80.645 73.66) (xy 78.105 71.12)
       )
     )
@@
     (polygon
       (pts
-        (xy 81.28 53.34) (xy 139.7 53.34) (xy 139.7 104.14) (xy 107.442 104.14) (xy 105.41 102.108)
+        (xy 78.105 53.34) (xy 141.605 53.34) (xy 141.605 104.14) (xy 107.442 104.14) (xy 105.41 102.108)
         (xy 105.41 98.171) (xy 107.061 96.52) (xy 120.65 96.52) (xy 121.92 95.25) (xy 118.11 91.44)
         (xy 116.84 90.17) (xy 114.3 87.63) (xy 113.03 86.36) (xy 113.03 73.66) (xy 102.87 73.66)
-        (xy 83.82 73.66) (xy 81.28 71.12)
+        (xy 80.645 73.66) (xy 78.105 71.12)
       )
     )
