File: swd_shifter/swd_shifter.kicad_pcb (KiCad board)
At the start: 2 copper layers, 27.9 x 15.9 mm, 10 parts, among them J1 JTAG_STLINKV2, J2 PACKET_TRACE_PORT, J3 JTAG_10_PIN, U1 PCA9306

Commit message: [swd_shifter] Add SWO line conversion from target to host.
Parts:
- added Q1: BSS138, TO_SOT_Packages_SMD:SOT-23_Handsoldering, F.Cu at (161.8, 102.0)
- added R6: 10k, Resistors_SMD:R_0805_HandSoldering, F.Cu at (161.4, 97.5)
- added R7: 10k, Resistors_SMD:R_0805_HandSoldering, F.Cu at (161.2, 105.4)
Connections:
- net Net-(J1-Pad15) renamed /NRST
- net Net-(J1-Pad7) renamed /ST_SDA
- net Net-(J1-Pad9) renamed /ST_SCL
- net Net-(J2-Pad6) renamed /T_SCL
- net Net-(J2-Pad7) renamed /T_SDA
- C1 pad 1: Net-(C1-Pad1) -> 3V3
- J1 pad 1: Net-(J1-Pad1) -> /VREF
- J1 pad 13: Net-(J1-Pad13) -> ST_SWO
- J1 pad 2: Net-(J1-Pad1) -> /VREF
- J2 pad 1: Net-(J1-Pad1) -> VCC
- J2 pad 2: Net-(J2-Pad2) -> T_SWO
- J3 pad 1: Net-(J1-Pad1) -> VCC
- J3 pad 6: Net-(J3-Pad6) -> T_SWO
- R1 pad 2: Net-(C1-Pad1) -> /EN
- R4 pad 1: Net-(J1-Pad1) -> VCC
- R5 pad 1: Net-(J1-Pad1) -> VCC
- U1 pad 2: Net-(J1-Pad1) -> VCC
- U1 pad 7: Net-(C1-Pad1) -> 3V3
- U1 pad 8: Net-(C1-Pad1) -> /EN
Routing:
- net VCC: track 0.00 -> 51.4 mm, vias 0 -> 4
- net Net-(J1-Pad1): track 35.7 -> 0.00 mm, vias 3 -> 0
- net T_SWO: track 0.00 -> 25.6 mm
- net 3V3: track 16.1 -> 30.8 mm
- net ST_SWO: track 0.00 -> 10.7 mm
- net Net-(C1-Pad1): track 9.11 -> 0.00 mm
- net /VREF: track 0.00 -> 5.11 mm, vias 0 -> 1
- net /EN: track 0.00 -> 3.81 mm
- net /ST_SCL: track 12.1 -> 11.4 mm
